Commit message: Added initial FastDDS framework

File: src/arm_description/urdf/arm.urdf.xacro (robot description, xacro)
@@ -10,6 +10,6 @@
             <box size="${box} ${box} ${box}"/>
         </geometry>
-        <material name="blue">
-            <color rgba = "0 0 1 1"/>
+        <material name="light gray">
+            <color rgba = "0.5 0.5 0.5 1"/>
         </material>
     </visual>
@@ -28,6 +28,6 @@
             <box size="${link} ${link} ${box}"/>
         </geometry>
-        <material name="red">
-            <color rgba = "1 0 0 1"/>
+        <material name="gray">
+            <color rgba = "0.4 0.4 0.4 1"/>
         </material>
     </visual>
@@ -64,6 +64,6 @@
             <box size="${link} ${link} ${box}"/>
         </geometry>
-        <material name="red">
-            <color rgba = "1 0 0 1"/>
+        <material name="gay">
+            <color rgba = "0.4 0.4 0.4 1"/>
         </material>
     </visual>
@@ -100,6 +100,6 @@
             <box size="${link} ${link} ${box}"/>
         </geometry>
-        <material name="red">
-            <color rgba = "1 0 0 1"/>
+        <material name="gray">
+            <color rgba = "0.4 0.4 0.4 1"/>
         </material>
     </visual>
